Commit message: feat: implement box lifting with kinematic grab + fix fork geometry
URDF changes:
- Lowered fork_lift_joint origin (0.175→0.150 m) so tines rest at
  ground level at joint=0 instead of floating 2.5 cm above
- Extended lower limit to -0.025 m so operator can fully lower forks
- Raised velocity_limit to 2.0 m/s

Kinematic grab (forklift_env._update_box_grab):
- Detects box 0.5–2.2 m forward, ±0.5 m lateral of forklift
- Raise command while in zone: attaches box kinematically to forks
- While carried: box position tracks fork tine height each step
- Fork lowers to ground (joint < 0.03): releases box at current position
- Prints [GRAB] / [DROP] events to terminal

Teleop: status line now shows [CARRYING] when box is on forks

Note: forklift.usd is git-ignored; reconvert with:
  ./isaaclab.sh -p scripts/tools/convert_urdf.py assets/forklift/forklift.urdf assets/forklift/forklift.usd --fix-base

Co-Authored-By: Claude Sonnet 4.6 <noreply@anthropic.com>

File: assets/forklift/forklift.urdf (robot description, URDF)
Before this commit: robot forklift, 9 links, 8 joints
Joints:
- joint fork_lift_joint: limit lower=0.0 upper=1.5 effort=5000.0 velocity=0.5 -> lower=-0.025 upper=1.5 effort=5000.0 velocity=2.0; origin xyz=0.05 0 0.175 rpy=0 0 0 -> xyz=0.05 0 0.150 rpy=0 0 0

Commit message: fix: resolve articulation crash by reconverting URDF without --fix-base
The previous USD (converted with --fix-base) created a PhysicsFixedJoint
called root_joint at z=0, while init_state.pos=(0,0,0.3) placed the robot
at z=0.3.  PhysX rejected this as "disjointed body transforms" and refused
to create the articulation.

Fix: reconvert the URDF without --fix-base so ArticulationRootAPI is applied
directly to base_link with no fixed root joint.  The robot is driven via root
velocity, so a fixed base joint was never needed.

Verified: simulation starts cleanly, all 5 joints found, 18 obstacle boxes
placed, "Forklift Teleoperation Ready" prints and steps run successfully.

Co-Authored-By: Claude Sonnet 4.6 <noreply@anthropic.com>

File: assets/forklift/forklift.urdf (robot description, URDF)
Before this commit: robot forklift, 9 links, 8 joints
Joints:
- joint fork_lift_joint: limit lower=-0.025 upper=1.5 effort=5000.0 velocity=2.0 -> lower=0.0 upper=1.5 effort=5000.0 velocity=2.0
