Commit message: Fixed some bugs

File: assets/forklift/forklift.urdf (robot description, URDF)
Before this commit: robot forklift, 9 links, 8 joints
Links:
- link base_link: geometry collision box size=1.8 1.0 0.6; visual mesh filename=../48-forklift/Forklift.obj scale=0.004 0.004 0.004
- link front_left_caster: geometry collision sphere radius=0.2
- link front_right_caster: geometry collision sphere radius=0.2
- link mast: geometry collision box size=0.15 0.8 1.8
- link rear_left_wheel: geometry collision cylinder length=0.15 radius=0.3
- link rear_right_wheel: geometry collision cylinder length=0.15 radius=0.3
