Commit message: heavy_machines: 8 more machines; review-driven fixes to checks, env, tasks
Machines (each built, adversarially reviewed against the real class and
its renders, then fixed): mini excavator, wheeled excavator, rigid haul
truck, motor grader, single-drum soil compactor, tracked asphalt paver,
3-axle concrete mixer truck, telescopic boom lift.

Fixes from the reviews:
- hydraulic_excavator: backhoe bucket (curl pulls the teeth toward the
  machine; it was a face shovel), front camera moved out of the opaque cab.
- render: painter's order was inverted for every view.
- checks: follower init/limit consistency, left/right by accumulated
  rotation (prismatic: sideways travel), overlap sweep over every tool
  range and full steering lock, camera inside/blocked, tool visibility.
- env: speed-dependent steering/articulation limit (max_lat_accel).
- tasks: readable instructions ('extend the stick', 'swing the chute
  left'), range-relative stop tolerance, capped scripted speeds, steering
  re-centred after turns, per-joint timeouts.
- tests: unwrapped yaw, slow tools get enough time, lateral-accel test.

Co-Authored-By: Claude Opus 5.5 <noreply@anthropic.com>
Claude-Session: https://claude.ai/code/session_01JLcQ8prorSGEwEdaSRwGcu

File: assets/heavy_machines/hydraulic_excavator/hydraulic_excavator.urdf (robot description, URDF)
Before this commit: robot hydraulic_excavator, 7 links, 6 joints
Links:
- link bucket: geometry collision box size=0.335261 1.2 0.06; collision box size=0.428019 1.2 0.06
Joints:
- joint bucket_joint: axis 0 -1 0 -> 0 1 0
