Commit message: heavy_machines: fix env issues from the Isaac Lab API review; final batch fixes
Env (each verified against the Isaac Lab source in this repo):
- URDF limits padded by 1e-4 (written at full precision): Isaac Lab rejects
  default joint positions outside the float32/degree PhysX limits, and many
  joints start exactly on a limit (mini excavator blade could not load).
- Pose is authoritative: PhysX now gets zero root/joint velocities, so it no
  longer advances the machine one substep past its cameras (true velocities
  are reported as obs['joint_vel'] and obs['base_twist_body']).
- Cameras refresh every control step (a 15 Hz period drifted in float32 and
  repeated frames); 3 re-renders after reset so episodes don't start on the
  previous scene.
- URDF->USD conversion cached next to the URDF (was re-imported into /tmp
  on every launch); props get a parent Xform.
- Per-wheel rolling speed (inner/outer, steered, articulated rear frame);
  actual joint velocities for steering, tools at limits and followers.
- Props moved outside the scripted work area (the machine passes through
  them); turn semantics in reverse documented.
- Scripts honour --device; teleop chase camera + real-time pacing; demo uses
  env.step_dt and realistic speeds; showcase spaces machines by swept extent;
  collector odometry twist in the root frame.
- Tests: no side slip at the axles, wheels roll at ground speed.

Also the remaining review fixes for backhoe loader, crane, telehandler and
scraper.

Co-Authored-By: Claude Opus 5.5 <noreply@anthropic.com>
Claude-Session: https://claude.ai/code/session_01JLcQ8prorSGEwEdaSRwGcu

File: assets/heavy_machines/articulated_dump_truck/articulated_dump_truck.urdf (robot description, URDF)
Before this commit: robot articulated_dump_truck, 13 links, 12 joints
Joints:
- joint articulation_joint: limit lower=-0.785 upper=0.785 effort=10000000 velocity=0.35 -> lower=-0.7851 upper=0.7851 effort=10000000 velocity=0.35
- joint dump_joint: limit lower=0 upper=1.22 effort=10000000 velocity=0.1 -> lower=-0.0001 upper=1.2201 effort=10000000 velocity=0.1
- joint left_hoist_barrel_joint: limit lower=0.141874 upper=0.686772 effort=10000000 velocity=0.12827 -> lower=0.141774023 upper=0.68687242 effort=10000000 velocity=0.12827
- joint left_hoist_rod_joint: limit lower=-0.05 upper=2.355651 effort=10000000 velocity=0.288988 -> lower=-0.0501 upper=2.35575076 effort=10000000 velocity=0.288988
- joint right_hoist_barrel_joint: limit lower=0.141874 upper=0.686772 effort=10000000 velocity=0.12827 -> lower=0.141774023 upper=0.68687242 effort=10000000 velocity=0.12827
- joint right_hoist_rod_joint: limit lower=-0.05 upper=2.355651 effort=10000000 velocity=0.288988 -> lower=-0.0501 upper=2.35575076 effort=10000000 velocity=0.288988

File: assets/heavy_machines/asphalt_paver/asphalt_paver.urdf (robot description, URDF)
Before this commit: robot asphalt_paver, 10 links, 9 joints
Joints:
- joint left_extension_joint: limit lower=0 upper=1.225 effort=10000000 velocity=0.15 -> lower=-0.0001 upper=1.2251 effort=10000000 velocity=0.15
- joint left_wing_joint: limit lower=0 upper=1.15 effort=10000000 velocity=0.25 -> lower=-0.0001 upper=1.1501 effort=10000000 velocity=0.25
- joint lift_cylinder_joint: limit lower=-1.765719 upper=-1.623177 effort=10000000 velocity=1 -> lower=-1.76581946 upper=-1.62307685 effort=10000000 velocity=1
- joint right_extension_joint: limit lower=0 upper=1.225 effort=10000000 velocity=0.15 -> lower=-0.0001 upper=1.2251 effort=10000000 velocity=0.15
- joint right_wing_joint: limit lower=0 upper=1.15 effort=10000000 velocity=0.25 -> lower=-0.0001 upper=1.1501 effort=10000000 velocity=0.25
- joint screed_lift_joint: limit lower=0 upper=0.279482 effort=10000000 velocity=0.079852 -> lower=-0.0001 upper=0.279581773 effort=10000000 velocity=0.079852
- joint tow_arm_joint: limit lower=0 upper=0.09 effort=10000000 velocity=0.025714 -> lower=-0.0001 upper=0.0901 effort=10000000 velocity=0.025714

File: assets/heavy_machines/backhoe_loader/backhoe_loader.urdf (robot description, URDF)
Before this commit: robot backhoe_loader, 22 links, 21 joints
Links:
- link boom: geometry collision box size=1.005684 0.3 0.36; collision box size=1.438367 0.26 0.3
- link boom_cylinder: geometry visual cylinder length=0.07 radius=0.1003; visual cylinder length=0.187 radius=0.08075
- link boom_rod: geometry visual cylinder length=0.14 radius=0.075; visual cylinder length=0.614633 radius=0.05
- link chassis: geometry collision box size=0.1 0.5 0.1; collision box size=0.1 0.5 0.3
- link dipper_rod: geometry visual cylinder length=0.126 radius=0.0675; visual cylinder length=0.763784 radius=0.045
- link lift_cylinders: geometry visual cylinder length=0.07 radius=0.0885; visual cylinder length=0.07 radius=0.0885
- link lift_rods: geometry visual cylinder length=0.126 radius=0.0675; visual cylinder length=0.126 radius=0.0675
- link loader_arm: geometry collision box size=0.30377 0.14 0.26; collision box size=0.30377 0.14 0.26
Joints:
- joint backhoe_bucket_joint: limit lower=-1.1 upper=2.45 effort=10000000 velocity=1.5 -> lower=-1.1001 upper=2.4501 effort=10000000 velocity=1.5
- joint boom_cylinder_joint: limit lower=-1.071027 upper=1.071027 effort=10000000 velocity=0.89926 -> lower=-1.29748251 upper=1.29748251 effort=10000000 velocity=1.071394; origin xyz=0.05 0 -0.2 rpy=0 -0.253505 0 -> xyz=0.28 0 -0.15 rpy=0 -0.249018 0
- joint boom_joint: limit lower=-1.15 upper=1.48 effort=10000000 velocity=1 -> lower=-1.1501 upper=1.4801 effort=10000000 velocity=1
- joint boom_rod_joint: limit lower=-0.283973 upper=0.283973 effort=10000000 velocity=0.30074 -> lower=-0.057717493 upper=0.057717493 effort=10000000 velocity=0.128606; origin xyz=0.9 0 -0.05 rpy=0 -3.230098 0 -> xyz=1.25 0 0 rpy=0 -3.225611 0
- joint dipper_cylinder_joint: limit lower=-0.103506 upper=0.103506 effort=10000000 velocity=0.169588 -> lower=-0.0736522921 upper=0.0736522921 effort=10000000 velocity=0.151002; origin xyz=0.95 0 0.55 rpy=0 0.251294 0 -> xyz=0.95 0 0.55 rpy=0 0.231793 0
- joint dipper_rod_joint: limit lower=-1.136494 upper=1.136494 effort=10000000 velocity=1.030412 -> lower=-1.01654771 upper=1.01654771 effort=10000000 velocity=1.048998; origin xyz=-0.3 0 0.1 rpy=0 -4.690299 0 -> xyz=-0.3 0 0.1 rpy=0 -4.559799 0
- joint front_left_steer_joint: limit lower=-0.8 upper=0.8 effort=10000000 velocity=1 -> lower=-0.8001 upper=0.8001 effort=10000000 velocity=1
- joint front_right_steer_joint: limit lower=-0.8 upper=0.8 effort=10000000 velocity=1 -> lower=-0.8001 upper=0.8001 effort=10000000 velocity=1
- joint left_stabilizer_joint: limit lower=0 upper=0.45 effort=10000000 velocity=0.25 -> lower=-0.0001 upper=0.4501 effort=10000000 velocity=0.25
- joint lift_cylinder_joint: limit lower=-0.45801 upper=0.45801 effort=10000000 velocity=0.279635 -> lower=-0.0303205454 upper=0.0303205454 effort=10000000 velocity=0.104346; origin xyz=2.57 0 0.15 rpy=0 -2.652327 0 -> xyz=2.42 0 -0.02 rpy=0 -2.220435 0
- joint lift_rod_joint: limit lower=-1.18951 upper=1.18951 effort=10000000 velocity=0.579635 -> lower=-0.818879455 upper=0.818879455 effort=10000000 velocity=0.439654; origin xyz=0.3 0 -0.7 rpy=0 -5.10242 0 -> xyz=0.4 0 0 rpy=0 -4.593028 0
- joint loader_arm_joint: limit lower=-0.04 upper=1.423 effort=10000000 velocity=0.3 -> lower=-0.0401 upper=1.5781 effort=10000000 velocity=0.344; origin xyz=1 0 0.98 rpy=0 0 0 -> xyz=1.24 0 0.98 rpy=0 0 0
- joint loader_bucket_joint: limit lower=-0.95 upper=0.75 effort=10000000 velocity=1.15 -> lower=-0.9501 upper=0.7501 effort=10000000 velocity=1.15
- joint right_stabilizer_joint: limit lower=0 upper=0.45 effort=10000000 velocity=0.25 -> lower=-0.0001 upper=0.4501 effort=10000000 velocity=0.25
- joint shovel_level_joint: limit lower=-0.7515 upper=0.7515 effort=10000000 velocity=0.4 -> lower=-0.8291 upper=0.8291 effort=10000000 velocity=0.444; origin xyz=1.93 0 -1.42 rpy=0 0.6915 0 -> xyz=1.69 0 -1.42 rpy=0 0.769 0
- joint stick_joint: limit lower=-1.45 upper=0.95 effort=10000000 velocity=1 -> lower=-1.1501 upper=0.9501 effort=10000000 velocity=1
- joint swing_joint: limit lower=-1.5 upper=1.5 effort=10000000 velocity=1 -> lower=-1.5001 upper=1.5001 effort=10000000 velocity=1

File: assets/heavy_machines/bulldozer/bulldozer.urdf (robot description, URDF)
Before this commit: robot bulldozer, 18 links, 17 joints
Joints:
- joint blade_lift_joint: limit lower=-0.161481 upper=0.359077 effort=10000000 velocity=0.18 -> lower=-0.161581292 upper=0.35917731 effort=10000000 velocity=0.18
- joint blade_tilt_joint: limit lower=-0.2 upper=0.2 effort=10000000 velocity=0.15 -> lower=-0.2001 upper=0.2001 effort=10000000 velocity=0.15
- joint left_brace_rod_joint: limit lower=-0.500925 upper=0.443577 effort=10000000 velocity=2 -> lower=-0.501025382 upper=0.443677319 effort=10000000 velocity=2
- joint left_push_arm_joint: limit lower=-0.150532 upper=0.150321 effort=10000000 velocity=2 -> lower=-0.150631716 upper=0.150420929 effort=10000000 velocity=2
- joint left_tilt_brace_joint: limit lower=-0.336773 upper=0.308225 effort=10000000 velocity=2 -> lower=-0.336873256 upper=0.308325241 effort=10000000 velocity=2
- joint lift_cylinder_joint: limit lower=-0.914184 upper=-0.303182 effort=10000000 velocity=2 -> lower=-0.914284385 upper=-0.303081521 effort=10000000 velocity=2
- joint lift_rod_joint: limit lower=2.379334 upper=2.48889 effort=10000000 velocity=2 -> lower=2.37923382 upper=2.48898956 effort=10000000 velocity=2
- joint right_push_arm_joint: limit lower=-0.150321 upper=0.150532 effort=10000000 velocity=2 -> lower=-0.150420929 upper=0.150631716 effort=10000000 velocity=2
- joint right_tilt_cylinder_joint: limit lower=-0.308326 upper=0.336875 effort=10000000 velocity=2 -> lower=-0.308425534 upper=0.336975461 effort=10000000 velocity=2
- joint right_tilt_rod_joint: limit lower=-0.442427 upper=0.499594 effort=10000000 velocity=2 -> lower=-0.442526921 upper=0.499694044 effort=10000000 velocity=2
- joint ripper_beam_joint: limit lower=-0.605388 upper=0.594724 effort=10000000 velocity=2 -> lower=-0.605487653 upper=0.594823722 effort=10000000 velocity=2
- joint ripper_cylinder_joint: limit lower=-0.927928 upper=0.024075 effort=10000000 velocity=2 -> lower=-0.928027997 upper=0.0241751097 effort=10000000 velocity=2
- joint ripper_joint: limit lower=-0.544724 upper=0.555388 effort=10000000 velocity=0.3 -> lower=-0.544823722 upper=0.555487653 effort=10000000 velocity=0.3
- joint ripper_link_joint: limit lower=-0.594724 upper=0.605388 effort=10000000 velocity=2 -> lower=-0.594823722 upper=0.605487653 effort=10000000 velocity=2
- joint ripper_rod_joint: limit lower=-0.024075 upper=0.927928 effort=10000000 velocity=2 -> lower=-0.0241751097 upper=0.928027997 effort=10000000 velocity=2

File: assets/heavy_machines/compact_track_loader/compact_track_loader.urdf (robot description, URDF)
Before this commit: robot compact_track_loader, 7 links, 6 joints
Joints:
- joint bucket_joint: limit lower=-1.8 upper=0.55 effort=10000000 velocity=1 -> lower=-1.8001 upper=0.5501 effort=10000000 velocity=1
- joint lift_arm_joint: limit lower=-0.02 upper=1.06 effort=10000000 velocity=0.32 -> lower=-0.0201 upper=1.0601 effort=10000000 velocity=0.32
- joint lift_cylinder_joint: limit lower=0.750563 upper=1.401355 effort=10000000 velocity=1 -> lower=0.750462557 upper=1.401455 effort=10000000 velocity=1
- joint lift_rod_joint: limit lower=-2.900238 upper=-2.27103 effort=10000000 velocity=1 -> lower=-2.90033766 upper=-2.2709301 effort=10000000 velocity=1

File: assets/heavy_machines/concrete_mixer_truck/concrete_mixer_truck.urdf (robot description, URDF)
Before this commit: robot concrete_mixer_truck, 19 links, 18 joints
Joints:
- joint chute_lift_barrel_joint: limit lower=0.055251 upper=0.595318 effort=10000000 velocity=0.188908 -> lower=0.0551505636 upper=0.595417944 effort=10000000 velocity=0.188908
- joint chute_lift_joint: limit lower=-0.55 upper=0.35 effort=10000000 velocity=0.25 -> lower=-0.5501 upper=0.3501 effort=10000000 velocity=0.25
- joint chute_lift_rod_joint: limit lower=-0.302181 upper=0.031962 effort=10000000 velocity=0.131706 -> lower=-0.302281083 upper=0.0320620602 effort=10000000 velocity=0.131706
- joint chute_swing_joint: limit lower=-1.55 upper=1.55 effort=10000000 velocity=0.3 -> lower=-1.5501 upper=1.5501 effort=10000000 velocity=0.3
- joint front_left_steer_joint: limit lower=-0.8 upper=0.8 effort=10000000 velocity=0.8 -> lower=-0.8001 upper=0.8001 effort=10000000 velocity=0.8
- joint front_right_steer_joint: limit lower=-0.8 upper=0.8 effort=10000000 velocity=0.8 -> lower=-0.8001 upper=0.8001 effort=10000000 velocity=0.8

File: assets/heavy_machines/hydraulic_excavator/hydraulic_excavator.urdf (robot description, URDF)
Before this commit: robot hydraulic_excavator, 7 links, 6 joints
Joints:
- joint boom_joint: limit lower=-0.9 upper=1 effort=10000000 velocity=0.55 -> lower=-0.9001 upper=1.0001 effort=10000000 velocity=0.55
- joint bucket_joint: limit lower=-1.2 upper=1.75 effort=10000000 velocity=1 -> lower=-1.2001 upper=1.7501 effort=10000000 velocity=1
- joint stick_joint: limit lower=-1.35 upper=0.9 effort=10000000 velocity=0.65 -> lower=-1.3501 upper=0.9001 effort=10000000 velocity=0.65

File: assets/heavy_machines/mini_excavator/mini_excavator.urdf (robot description, URDF)
Before this commit: robot mini_excavator, 19 links, 18 joints
Joints:
- joint arm_cyl_barrel_joint: limit lower=-0.077589 upper=0.077589 effort=10000000 velocity=0.101527 -> lower=-0.0776888836 upper=0.0776888836 effort=10000000 velocity=0.101527
- joint arm_cyl_rod_joint: limit lower=-0.912411 upper=0.912411 effort=10000000 velocity=0.848473 -> lower=-0.912511116 upper=0.912511116 effort=10000000 velocity=0.848473
- joint blade_cyl_barrel_joint: limit lower=-0.551507 upper=0.551507 effort=10000000 velocity=0.553786 -> lower=-0.551607269 upper=0.551607269 effort=10000000 velocity=0.553786
- joint blade_cyl_rod_joint: limit lower=-0.182248 upper=0.182248 effort=10000000 velocity=0.203786 -> lower=-0.182348038 upper=0.182348038 effort=10000000 velocity=0.203786
- joint blade_joint: limit lower=-0.390613 upper=0.347905 effort=10000000 velocity=0.35 -> lower=-0.390713215 upper=0.348005248 effort=10000000 velocity=0.35
- joint boom_cyl_barrel_joint: limit lower=-1.053015 upper=1.053015 effort=10000000 velocity=0.729615 -> lower=-1.05311505 upper=1.05311505 effort=10000000 velocity=0.729615
- joint boom_cyl_rod_joint: limit lower=-0.126985 upper=0.126985 effort=10000000 velocity=0.120385 -> lower=-0.127084951 upper=0.127084951 effort=10000000 velocity=0.120385
- joint boom_joint: limit lower=-1.16 upper=1.12 effort=10000000 velocity=0.75 -> lower=-1.1601 upper=1.1201 effort=10000000 velocity=0.75
- joint boom_swing_joint: limit lower=-1.05 upper=1.31 effort=10000000 velocity=0.45 -> lower=-1.0501 upper=1.3101 effort=10000000 velocity=0.45
- joint bucket_cyl_barrel_joint: limit lower=-0.150643 upper=0.150643 effort=10000000 velocity=0.156148 -> lower=-0.15074316 upper=0.15074316 effort=10000000 velocity=0.156148
- joint bucket_cyl_rod_joint: limit lower=-0.819882 upper=0.819882 effort=10000000 velocity=0.699905 -> lower=-0.81998248 upper=0.81998248 effort=10000000 velocity=0.699905
- joint bucket_dogbone_joint: limit lower=-0.950526 upper=0.950526 effort=10000000 velocity=0.806052 -> lower=-0.95062564 upper=0.95062564 effort=10000000 velocity=0.806052
- joint bucket_hlink_joint: limit lower=-1.068864 upper=1.068864 effort=10000000 velocity=0.902202 -> lower=-1.06896408 upper=1.06896408 effort=10000000 velocity=0.902202
- joint bucket_joint: limit lower=-1.05 upper=2.15 effort=10000000 velocity=1.3 -> lower=-1.0501 upper=2.1501 effort=10000000 velocity=1.3
- joint stick_joint: limit lower=-1.05 upper=0.85 effort=10000000 velocity=0.85 -> lower=-1.0501 upper=0.8501 effort=10000000 velocity=0.85

File: assets/heavy_machines/motor_grader/motor_grader.urdf (robot description, URDF)
Before this commit: robot motor_grader, 22 links, 21 joints
Joints:
- joint blade_lift_joint: limit lower=-0.14 upper=0.213 effort=10000000 velocity=0.1 -> lower=-0.1401 upper=0.2131 effort=10000000 velocity=0.1
- joint blade_rotate_joint: limit lower=-1.4 upper=1.4 effort=10000000 velocity=0.25 -> lower=-1.4001 upper=1.4001 effort=10000000 velocity=0.25
- joint blade_shift_joint: limit lower=-0.68 upper=0.68 effort=10000000 velocity=0.22 -> lower=-0.6801 upper=0.6801 effort=10000000 velocity=0.22
- joint front_left_steer_joint: limit lower=-0.83 upper=0.83 effort=10000000 velocity=0.8 -> lower=-0.8301 upper=0.8301 effort=10000000 velocity=0.8
- joint front_right_steer_joint: limit lower=-0.83 upper=0.83 effort=10000000 velocity=0.8 -> lower=-0.8301 upper=0.8301 effort=10000000 velocity=0.8
- joint left_lift_barrel_joint: limit lower=0.12822 upper=0.369273 effort=10000000 velocity=0.2 -> lower=0.128119625 upper=0.369372741 effort=10000000 velocity=0.2
- joint left_lift_eye_joint: limit lower=-0.263 upper=0.19 effort=10000000 velocity=0.2 -> lower=-0.2631 upper=0.1901 effort=10000000 velocity=0.2
- joint left_lift_rod_joint: limit lower=0.12822 upper=0.369273 effort=10000000 velocity=0.2 -> lower=0.128119625 upper=0.369372741 effort=10000000 velocity=0.2
- joint right_lift_barrel_joint: limit lower=-0.369273 upper=-0.12822 effort=10000000 velocity=0.2 -> lower=-0.369372741 upper=-0.128119625 effort=10000000 velocity=0.2
- joint right_lift_eye_joint: limit lower=-0.263 upper=0.19 effort=10000000 velocity=0.2 -> lower=-0.2631 upper=0.1901 effort=10000000 velocity=0.2
- joint right_lift_rod_joint: limit lower=-0.369273 upper=-0.12822 effort=10000000 velocity=0.2 -> lower=-0.369372741 upper=-0.128119625 effort=10000000 velocity=0.2
- joint ripper_joint: limit lower=-0.52 upper=0.675 effort=10000000 velocity=0.35 -> lower=-0.5201 upper=0.6751 effort=10000000 velocity=0.35
- joint ripper_toolbar_joint: limit lower=-0.725 upper=0.57 effort=10000000 velocity=0.45 -> lower=-0.7251 upper=0.5701 effort=10000000 velocity=0.45
- joint ripper_upper_link_joint: limit lower=-0.57 upper=0.725 effort=10000000 velocity=0.45 -> lower=-0.5701 upper=0.7251 effort=10000000 velocity=0.45

File: assets/heavy_machines/rigid_haul_truck/rigid_haul_truck.urdf (robot description, URDF)
Before this commit: robot rigid_haul_truck, 15 links, 14 joints
Joints:
- joint dump_body_joint: limit lower=0 upper=0.96 effort=10000000 velocity=0.096 -> lower=-0.0001 upper=0.9601 effort=10000000 velocity=0.096
- joint front_left_steer_joint: limit lower=-0.7 upper=0.7 effort=10000000 velocity=0.8 -> lower=-0.7001 upper=0.7001 effort=10000000 velocity=0.8
- joint front_right_steer_joint: limit lower=-0.7 upper=0.7 effort=10000000 velocity=0.8 -> lower=-0.7001 upper=0.7001 effort=10000000 velocity=0.8
- joint hoist_barrel_joint: limit lower=0.793505 upper=1.745207 effort=10000000 velocity=0.14117 -> lower=0.79340491 upper=1.74530668 effort=10000000 velocity=0.14117
- joint hoist_rod_joint: limit lower=-0.011723 upper=1.308912 effort=10000000 velocity=0.178063 -> lower=-0.0118226254 upper=1.30901153 effort=10000000 velocity=0.178063
- joint hoist_stage_joint: limit lower=-0.011723 upper=1.308912 effort=10000000 velocity=0.178063 -> lower=-0.0118226254 upper=1.30901153 effort=10000000 velocity=0.178063
