Commit message: heavy_machines: fix env issues from the Isaac Lab API review; final batch fixes
Env (each verified against the Isaac Lab source in this repo):
- URDF limits padded by 1e-4 (written at full precision): Isaac Lab rejects
  default joint positions outside the float32/degree PhysX limits, and many
  joints start exactly on a limit (mini excavator blade could not load).
- Pose is authoritative: PhysX now gets zero root/joint velocities, so it no
  longer advances the machine one substep past its cameras (true velocities
  are reported as obs['joint_vel'] and obs['base_twist_body']).
- Cameras refresh every control step (a 15 Hz period drifted in float32 and
  repeated frames); 3 re-renders after reset so episodes don't start on the
  previous scene.
- URDF->USD conversion cached next to the URDF (was re-imported into /tmp
  on every launch); props get a parent Xform.
- Per-wheel rolling speed (inner/outer, steered, articulated rear frame);
  actual joint velocities for steering, tools at limits and followers.
- Props moved outside the scripted work area (the machine passes through
  them); turn semantics in reverse documented.
- Scripts honour --device; teleop chase camera + real-time pacing; demo uses
  env.step_dt and realistic speeds; showcase spaces machines by swept extent;
  collector odometry twist in the root frame.
- Tests: no side slip at the axles, wheels roll at ground speed.

Also the remaining review fixes for backhoe loader, crane, telehandler and
scraper.

Co-Authored-By: Claude Opus 5.5 <noreply@anthropic.com>
Claude-Session: https://claude.ai/code/session_01JLcQ8prorSGEwEdaSRwGcu

File: assets/heavy_machines/rough_terrain_crane/rough_terrain_crane.urdf (robot description, URDF)
Before this commit: robot rough_terrain_crane, 25 links, 24 joints
Links:
- link boom_base: geometry collision box size=9.3 0.72 0.7; visual box size=0.1 0.06 0.08
- link boom_sec2: geometry collision box size=8.3 0.62 0.58; visual box size=0.12 0.69 0.04
- link boom_sec3: geometry collision box size=8.3 0.53 0.47; visual box size=0.12 0.6 0.04
- link boom_sec4: geometry collision box size=0.7 0.06 0.925; collision box size=0.7 0.06 0.925
- link carrier: geometry collision box size=0.12 2 0.28; collision box size=0.12 2 0.28
- link front_left_knuckle: geometry collision cylinder length=0.2 radius=0.15; visual cylinder length=0.2 radius=0.15
- link front_right_knuckle: geometry collision cylinder length=0.2 radius=0.15; visual cylinder length=0.2 radius=0.15
- link lift_cylinder: geometry visual cylinder length=0.14 radius=0.2; visual cylinder length=0.42 radius=0.14
- link lift_cylinder_rod: geometry visual cylinder length=0.36 radius=0.13; visual cylinder length=2.023547 radius=0.11
- link superstructure: geometry collision box size=0.6 1.6 0.3; collision box size=0.7 0.06 0.55
Joints:
- joint boom_luff_joint: limit lower=0 upper=1.35 effort=10000000 velocity=0.1 -> lower=-0.0001 upper=1.3501 effort=10000000 velocity=0.1
- joint boom_sec3_joint: limit lower=-0.01 upper=7.21 effort=10000000 velocity=0.55 -> lower=-0.0101 upper=7.2101 effort=10000000 velocity=0.55
- joint boom_sec4_joint: limit lower=-0.01 upper=7.21 effort=10000000 velocity=0.55 -> lower=-0.0101 upper=7.2101 effort=10000000 velocity=0.55
- joint boom_telescope_joint: limit lower=0 upper=7.2 effort=10000000 velocity=0.5 -> lower=-0.0001 upper=7.2001 effort=10000000 velocity=0.5
- joint front_left_steer_joint: limit lower=-0.7 upper=0.7 effort=10000000 velocity=0.6 -> lower=-0.7001 upper=0.7001 effort=10000000 velocity=0.6
- joint front_right_steer_joint: limit lower=-0.7 upper=0.7 effort=10000000 velocity=0.6 -> lower=-0.7001 upper=0.7001 effort=10000000 velocity=0.6
- joint hoist_joint: limit lower=0.8 upper=14 effort=10000000 velocity=1 -> lower=0.7999 upper=14.0001 effort=10000000 velocity=1
- joint hook_swivel_joint: limit lower=-1.36 upper=0.01 effort=10000000 velocity=0.15 -> lower=-1.3601 upper=0.0101 effort=10000000 velocity=0.15
- joint lift_cylinder_joint: limit lower=0.087617 upper=1.476257 effort=10000000 velocity=0.145455 -> lower=0.133352931 upper=1.43888568 effort=10000000 velocity=0.139284; origin xyz=-0.95 0 0.25 rpy=0 0 0 -> xyz=-1 0 0.05 rpy=0 0 0
- joint lift_cylinder_rod_joint: limit lower=0.026257 upper=0.187617 effort=10000000 velocity=0.054545 -> lower=-0.0113143203 upper=0.233552931 effort=10000000 velocity=0.060716; origin xyz=4.2 0 -0.5 rpy=0 0 0 -> xyz=3.2 0 -0.7 rpy=0 0 0
- joint rope_seg_1_joint: limit lower=0.715 upper=2.055 effort=10000000 velocity=0.15 -> lower=0.7149 upper=2.0551 effort=10000000 velocity=0.15
- joint rope_seg_2_joint: limit lower=0.715 upper=3.375 effort=10000000 velocity=0.25 -> lower=0.7149 upper=3.3751 effort=10000000 velocity=0.25
- joint rope_seg_3_joint: limit lower=0.715 upper=4.695 effort=10000000 velocity=0.35 -> lower=0.7149 upper=4.6951 effort=10000000 velocity=0.35
- joint rope_seg_4_joint: limit lower=0.715 upper=6.015 effort=10000000 velocity=0.45 -> lower=0.7149 upper=6.0151 effort=10000000 velocity=0.45
- joint rope_seg_5_joint: limit lower=0.715 upper=7.335 effort=10000000 velocity=0.55 -> lower=0.7149 upper=7.3351 effort=10000000 velocity=0.55
- joint rope_seg_6_joint: limit lower=0.715 upper=8.655 effort=10000000 velocity=0.65 -> lower=0.7149 upper=8.6551 effort=10000000 velocity=0.65
- joint rope_seg_7_joint: limit lower=0.715 upper=9.975 effort=10000000 velocity=0.75 -> lower=0.7149 upper=9.9751 effort=10000000 velocity=0.75
- joint rope_seg_8_joint: limit lower=0.715 upper=11.295 effort=10000000 velocity=0.85 -> lower=0.7149 upper=11.2951 effort=10000000 velocity=0.85
- joint rope_seg_9_joint: limit lower=0.715 upper=12.615 effort=10000000 velocity=0.95 -> lower=0.7149 upper=12.6151 effort=10000000 velocity=0.95

File: assets/heavy_machines/skid_steer_loader/skid_steer_loader.urdf (robot description, URDF)
Before this commit: robot skid_steer_loader, 11 links, 10 joints
Joints:
- joint bucket_joint: limit lower=-1.88 upper=0.55 effort=10000000 velocity=0.9 -> lower=-1.8801 upper=0.5501 effort=10000000 velocity=0.9
- joint lift_arm_joint: limit lower=0 upper=1.156251 effort=10000000 velocity=0.35 -> lower=-0.0001 upper=1.15635063 effort=10000000 velocity=0.35
- joint lift_cylinder_joint: limit lower=-0.346641 upper=0.346641 effort=10000000 velocity=2 -> lower=-0.346740802 upper=0.346740802 effort=10000000 velocity=2
- joint lift_rod_joint: limit lower=-0.271485 upper=0.271485 effort=10000000 velocity=2 -> lower=-0.271584512 upper=0.271584512 effort=10000000 velocity=2
- joint tilt_cylinder_joint: limit lower=-0.027257 upper=0.027257 effort=10000000 velocity=2 -> lower=-0.0273565783 upper=0.0273565783 effort=10000000 velocity=2
- joint tilt_rod_joint: limit lower=-0.173957 upper=0.173957 effort=10000000 velocity=2 -> lower=-0.17405654 upper=0.17405654 effort=10000000 velocity=2

File: assets/heavy_machines/soil_compactor/soil_compactor.urdf (robot description, URDF)
Before this commit: robot soil_compactor, 8 links, 7 joints
Joints:
- joint articulation_joint: limit lower=-0.593 upper=0.593 effort=10000000 velocity=0.3 -> lower=-0.5931 upper=0.5931 effort=10000000 velocity=0.3
- joint blade_cylinder_joint: limit lower=-0.291762 upper=0.291762 effort=10000000 velocity=0.314725 -> lower=-0.291861564 upper=0.291861564 effort=10000000 velocity=0.314725
- joint blade_cylinder_rod_joint: limit lower=-0.015657 upper=0.230489 effort=10000000 velocity=0.189341 -> lower=-0.0157567872 upper=0.23058856 effort=10000000 velocity=0.189341
- joint blade_joint: limit lower=-0.405 upper=0 effort=10000000 velocity=0.16 -> lower=-0.4051 upper=0.0001 effort=10000000 velocity=0.16

File: assets/heavy_machines/telehandler/telehandler.urdf (robot description, URDF)
Before this commit: robot telehandler, 15 links, 14 joints
Links:
- link boom_fly: geometry collision box size=0.15 0.4 0.15; collision box size=0.515667 0.4 0.33
- link carriage: geometry collision box size=0.06 0.12 1.04; collision box size=0.06 0.12 1.04
- link chassis: geometry collision box size=0.08 1.8 0.85; collision box size=0.14 1.7 0.16
- link front_left_knuckle: geometry collision cylinder length=0.25 radius=0.17; visual box size=0.04 0.03 0.3
- link front_right_knuckle: geometry collision cylinder length=0.25 radius=0.17; visual box size=0.04 0.03 0.3
- link lift_cylinder: geometry visual cylinder length=0.08 radius=0.16; visual cylinder length=0.3 radius=0.1
- link lift_rod: geometry visual cylinder length=0.24 radius=0.11; visual cylinder length=1.25123 radius=0.075
Joints:
- removed joint boom_fly_joint
- added joint boom_mid_1_joint: type prismatic, parent boom_base, child boom_mid_1, origin xyz=-0.1 0 0 rpy=0 0 0, axis 1 0 0, limit lower=-0.0001 upper=3.7331 effort=10000000 velocity=0.3
- joint boom_luff_joint: limit lower=-0.1269 upper=1.2086 effort=10000000 velocity=0.14 -> lower=-0.0479 upper=1.2086 effort=10000000 velocity=0.14
- joint boom_mid_2_joint: limit lower=0 upper=3.712 effort=10000000 velocity=0.3 -> lower=-0.0001 upper=7.4661 effort=10000000 velocity=0.6; origin xyz=0.1 0 0 rpy=0 0 0 -> xyz=0 0 0 rpy=0 0 0; parent boom_mid_1 -> boom_base
- joint boom_telescope_joint: child boom_mid_1 -> boom_fly; limit lower=0 upper=3.712 effort=10000000 velocity=0.3 -> lower=-0.0001 upper=11.1991 effort=10000000 velocity=0.9; origin xyz=-0.1 0 0 rpy=0 0 0 -> xyz=0.1 0 0 rpy=0 0 0
- joint carriage_level_joint: limit lower=-1.2586 upper=0.1769 effort=10000000 velocity=0.14 -> lower=-1.2586 upper=0.0979 effort=10000000 velocity=0.14; origin xyz=5.528244 0 -0.3 rpy=0 0 0 -> xyz=5.465667 0 -0.3 rpy=0 0 0
- joint fork_tilt_joint: limit lower=-1.25 upper=0.4 effort=10000000 velocity=0.45 -> lower=-0.9501 upper=0.4001 effort=10000000 velocity=0.45
- joint front_left_steer_joint: limit lower=-0.85 upper=0.85 effort=10000000 velocity=1 -> lower=-0.8501 upper=0.8501 effort=10000000 velocity=1
- joint front_right_steer_joint: limit lower=-0.85 upper=0.85 effort=10000000 velocity=1 -> lower=-0.8501 upper=0.8501 effort=10000000 velocity=1
- joint lift_cylinder_joint: limit lower=-0.659516 upper=0.659516 effort=10000000 velocity=0.18408 -> lower=-0.614539092 upper=0.614539092 effort=10000000 velocity=0.182487; origin xyz=-0.9 -0.12 0.345 rpy=0 -0.663234 0 -> xyz=-0.9 -0.12 0.345 rpy=0 -0.704678 0
- joint lift_rod_joint: limit lower=-0.048234 upper=0.048234 effort=10000000 velocity=0.05592 -> lower=-0.0538109081 upper=0.0538109081 effort=10000000 velocity=0.057513; origin xyz=2.9 0 -0.4 rpy=0 -3.263977 0 -> xyz=2.9 0 -0.4 rpy=0 -3.26592 0

File: assets/heavy_machines/telescopic_boom_lift/telescopic_boom_lift.urdf (robot description, URDF)
Before this commit: robot telescopic_boom_lift, 17 links, 16 joints
Joints:
- joint boom_joint: limit lower=0 upper=1.308997 effort=10000000 velocity=0.11 -> lower=-0.0001 upper=1.30909694 effort=10000000 velocity=0.11
- joint fly_joint: limit lower=0 upper=4.585 effort=10000000 velocity=0.36 -> lower=-0.0001 upper=4.5851 effort=10000000 velocity=0.36
- joint jib_joint: limit lower=-1.134464 upper=1.22173 effort=10000000 velocity=0.2 -> lower=-1.13456401 upper=1.22183048 effort=10000000 velocity=0.2
- joint jib_level_joint: limit lower=-1.358997 upper=0.05 effort=10000000 velocity=0.11 -> lower=-1.35909694 upper=0.0501 effort=10000000 velocity=0.11
- joint lift_cylinder_joint: limit lower=0.044317 upper=1.46992 effort=10000000 velocity=0.152992 -> lower=0.0442169795 upper=1.47002036 effort=10000000 velocity=0.152992
- joint platform_level_joint: limit lower=-1.27173 upper=1.184464 effort=10000000 velocity=0.2 -> lower=-1.27183048 upper=1.18456401 effort=10000000 velocity=0.2
- joint platform_rotate_joint: limit lower=-1.396263 upper=1.396263 effort=10000000 velocity=0.25 -> lower=-1.3963634 upper=1.3963634 effort=10000000 velocity=0.25
- joint rear_left_steer_joint: limit lower=-0.7 upper=0.7 effort=10000000 velocity=0.6 -> lower=-0.7001 upper=0.7001 effort=10000000 velocity=0.6
- joint rear_right_steer_joint: limit lower=-0.7 upper=0.7 effort=10000000 velocity=0.6 -> lower=-0.7001 upper=0.7001 effort=10000000 velocity=0.6
- joint telescope_joint: limit lower=0 upper=4.585 effort=10000000 velocity=0.36 -> lower=-0.0001 upper=4.5851 effort=10000000 velocity=0.36

File: assets/heavy_machines/wheel_loader/wheel_loader.urdf (robot description, URDF)
Before this commit: robot wheel_loader, 19 links, 18 joints
Joints:
- joint articulation_joint: limit lower=-0.7 upper=0.7 effort=10000000 velocity=0.35 -> lower=-0.7001 upper=0.7001 effort=10000000 velocity=0.35
- joint bucket_joint: limit lower=-1.13 upper=0.82 effort=10000000 velocity=1.15 -> lower=-1.1301 upper=0.8201 effort=10000000 velocity=1.15
- joint bucket_level_joint: limit lower=-0.541331 upper=0.541331 effort=10000000 velocity=0.272 -> lower=-0.541431181 upper=0.541431181 effort=10000000 velocity=0.272
- joint lift_arm_joint: limit lower=-0.03 upper=1.273328 effort=10000000 velocity=0.215 -> lower=-0.0301 upper=1.27342795 effort=10000000 velocity=0.215
- joint lift_cylinder_joint: limit lower=-0.389493 upper=0.389493 effort=10000000 velocity=0.221905 -> lower=-0.389593474 upper=0.389593474 effort=10000000 velocity=0.221905
- joint lift_rod_joint: limit lower=-0.302171 upper=0.302171 effort=10000000 velocity=0.193095 -> lower=-0.302270502 upper=0.302270502 effort=10000000 velocity=0.193095
- joint tilt_cylinder_joint: limit lower=-0.104825 upper=0.104825 effort=10000000 velocity=0.20005 -> lower=-0.104925 upper=0.104925 effort=10000000 velocity=0.20005
- joint tilt_cylinder_level_joint: limit lower=-0.560881 upper=0.560881 effort=10000000 velocity=0.27845 -> lower=-0.5609811 upper=0.5609811 effort=10000000 velocity=0.27845
- joint tilt_lever_joint: limit lower=-0.995 upper=0.995 effort=10000000 velocity=1.25 -> lower=-0.9951 upper=0.9951 effort=10000000 velocity=1.25
- joint tilt_lever_level_joint: limit lower=-0.541331 upper=0.541331 effort=10000000 velocity=0.272 -> lower=-0.541431181 upper=0.541431181 effort=10000000 velocity=0.272
- joint tilt_links_joint: limit lower=-0.995 upper=0.995 effort=10000000 velocity=1.25 -> lower=-0.9951 upper=0.9951 effort=10000000 velocity=1.25
- joint tilt_links_level_joint: limit lower=-0.541331 upper=0.541331 effort=10000000 velocity=0.272 -> lower=-0.541431181 upper=0.541431181 effort=10000000 velocity=0.272
- joint tilt_rod_joint: limit lower=-0.910175 upper=0.910175 effort=10000000 velocity=1.14995 -> lower=-0.910275 upper=0.910275 effort=10000000 velocity=1.14995
- joint tilt_rod_level_joint: limit lower=-0.430548 upper=0.430548 effort=10000000 velocity=0.23545 -> lower=-0.430648305 upper=0.430648305 effort=10000000 velocity=0.23545

File: assets/heavy_machines/wheel_tractor_scraper/wheel_tractor_scraper.urdf (robot description, URDF)
Before this commit: robot wheel_tractor_scraper, 15 links, 14 joints
Links:
- link hitch: geometry collision box size=0.505 0.7 0.55; collision cylinder length=0.6 radius=0.24
- link tractor: geometry collision box size=0.2 1.3 0.3; collision box size=0.25 1.4 0.95
Joints:
- joint apron_joint: limit lower=0 upper=0.55 effort=10000000 velocity=0.3 -> lower=-0.0001 upper=0.5501 effort=10000000 velocity=0.3
- joint bowl_joint: limit lower=-0.194112 upper=0 effort=10000000 velocity=0.09 -> lower=-0.194212434 upper=0.0001 effort=10000000 velocity=0.09
- joint ejector_joint: limit lower=0 upper=2.1 effort=10000000 velocity=0.35 -> lower=-0.0001 upper=2.1001 effort=10000000 velocity=0.35
- joint ejector_stage_joint: limit lower=-0.02 upper=1.07 effort=10000000 velocity=0.225 -> lower=-0.0201 upper=1.0701 effort=10000000 velocity=0.225
- joint gooseneck_pitch_joint: limit lower=-0.019889 upper=0.067855 effort=10000000 velocity=0.072136 -> lower=-0.0199886413 upper=0.0679549372 effort=10000000 velocity=0.072136
- joint left_lift_barrel_joint: limit lower=-0.042793 upper=0.150021 effort=10000000 velocity=0.093033 -> lower=-0.0428926545 upper=0.150121401 effort=10000000 velocity=0.093033
- joint left_lift_rod_joint: limit lower=-0.05 upper=0.597417 effort=10000000 velocity=0.303809 -> lower=-0.0501 upper=0.597516837 effort=10000000 velocity=0.303809
- joint right_lift_barrel_joint: limit lower=-0.042793 upper=0.150021 effort=10000000 velocity=0.093033 -> lower=-0.0428926545 upper=0.150121401 effort=10000000 velocity=0.093033
- joint right_lift_rod_joint: limit lower=-0.05 upper=0.597417 effort=10000000 velocity=0.303809 -> lower=-0.0501 upper=0.597516837 effort=10000000 velocity=0.303809
- joint steering_hitch_joint: limit lower=-0.9 upper=0.9 effort=10000000 velocity=0.4 -> lower=-0.9001 upper=0.9001 effort=10000000 velocity=0.4

File: assets/heavy_machines/wheeled_excavator/wheeled_excavator.urdf (robot description, URDF)
Before this commit: robot wheeled_excavator, 18 links, 17 joints
Joints:
- joint blade_joint: limit lower=-0.65 upper=0.15 effort=10000000 velocity=0.32 -> lower=-0.6501 upper=0.1501 effort=10000000 velocity=0.32
- joint boom_cylinder_joint: limit lower=-0.658278 upper=1.577987 effort=10000000 velocity=0.646315 -> lower=-0.658377945 upper=1.57808679 effort=10000000 velocity=0.646315
- joint boom_joint: limit lower=-1 upper=1.05 effort=10000000 velocity=0.55 -> lower=-1.0001 upper=1.0501 effort=10000000 velocity=0.55
- joint bucket_joint: limit lower=-1.1 upper=1.9 effort=10000000 velocity=1 -> lower=-1.1001 upper=1.9001 effort=10000000 velocity=1
- joint front_left_steer_joint: limit lower=-0.7 upper=0.7 effort=10000000 velocity=0.8 -> lower=-0.7001 upper=0.7001 effort=10000000 velocity=0.8
- joint front_right_steer_joint: limit lower=-0.7 upper=0.7 effort=10000000 velocity=0.8 -> lower=-0.7001 upper=0.7001 effort=10000000 velocity=0.8
- joint stick_cylinder_joint: limit lower=-2.870342 upper=-0.574783 effort=10000000 velocity=0.748625 -> lower=-2.8704416 upper=-0.574682617 effort=10000000 velocity=0.748625
- joint stick_joint: limit lower=-1.3 upper=0.8 effort=10000000 velocity=0.65 -> lower=-1.3001 upper=0.8001 effort=10000000 velocity=0.65
