Commit message: heavy_machines: finish fleet polish — every tool visible, no motion clashes, detailed reference excavator
- hydraulic_excavator: visual upgrade (track rollers/idlers/lugs, cab
  details, handrails, grille, shaped counterweight, boom/stick/bucket
  hydraulic cylinders as follower links); datasheet dims, joints, ranges
  and signs unchanged.
- motor_grader: moldboard clears the rear frame over the whole circle
  range; rear-facing camera shows the ripper.
- wheeled_excavator: folded bucket clears the boom; rear deck camera shows
  the stabiliser blade (moved aft so the counterweight facet doesn't fill
  a seventh of the frame at the near clip).
- backhoe_loader: roading length within 10% of the CAT 420 / JCB 3CX
  datasheet; folded backhoe clears chassis and stabilisers across the
  swing; loader carried 0.12 m above ground.
- asphalt_paver: side camera on the platform edge instead of floating
  0.15 m outboard.
- README: generated fleet table (check_machine.py --readme).

All 18 machines pass every check; offline suites pass (machines, env
control logic, ROS 2 bag round trip).

Co-Authored-By: Claude Opus 5.5 <noreply@anthropic.com>
Claude-Session: https://claude.ai/code/session_01JLcQ8prorSGEwEdaSRwGcu

File: assets/heavy_machines/backhoe_loader/backhoe_loader.urdf (robot description, URDF)
Before this commit: robot backhoe_loader, 22 links, 21 joints
Links:
- link boom: geometry collision box size=1.005684 0.3 0.36; collision box size=1.535871 0.26 0.3
- link chassis: geometry collision box size=0.1 0.5 0.3; collision box size=0.2 2.1 0.36
Joints:
- joint boom_cylinder_joint: origin xyz=0.28 0 -0.15 rpy=0 -0.249018 0 -> xyz=0.14 0 -0.15 rpy=0 -0.249018 0
- joint boom_joint: origin xyz=0.24 0 0.05 rpy=0 0 0 -> xyz=0.1 0 0.05 rpy=0 0 0
- joint dipper_cylinder_joint: origin xyz=0.95 0 0.55 rpy=0 0.231793 0 -> xyz=1.05 0 0.55 rpy=0 0.231793 0
- joint lift_cylinder_joint: limit lower=-0.0303205454 upper=0.0303205454 effort=10000000 velocity=0.104346 -> lower=-0.025167764 upper=0.025167764 effort=10000000 velocity=0.102155; origin xyz=2.42 0 -0.02 rpy=0 -2.220435 0 -> xyz=2.42 0 -0.02 rpy=0 -2.226653 0
- joint lift_rod_joint: limit lower=-0.818879455 upper=0.818879455 effort=10000000 velocity=0.439654 -> lower=-0.834167764 upper=0.834167764 effort=10000000 velocity=0.446155; origin xyz=0.4 0 0 rpy=0 -4.593028 0 -> xyz=0.4 0 0 rpy=0 -4.599245 0
- joint stick_joint: origin xyz=2.35 0 0 rpy=0 1.55 0 -> xyz=2.45 0 0 rpy=0 1.55 0
- joint swing_joint: limit lower=-1.5001 upper=1.5001 effort=10000000 velocity=1 -> lower=-1.4201 upper=1.4201 effort=10000000 velocity=1

File: assets/heavy_machines/hydraulic_excavator/hydraulic_excavator.urdf (robot description, URDF)
Before this commit: robot hydraulic_excavator, 7 links, 6 joints
Links:
- added link arm_cyl_barrel, mass 150; visual box size=0.126 0.105 0.084; visual box size=0.126 0.105 0.084
- added link arm_cyl_rod, mass 80; visual cylinder length=0.21 radius=0.07875; visual cylinder length=0.661339 radius=0.05775
- added link boom_cyl_barrel, mass 240; visual box size=0.12 0.1 0.08; visual box size=0.12 0.1 0.08
- added link boom_cyl_rod, mass 110; visual cylinder length=0.2 radius=0.075; visual cylinder length=0.2 radius=0.075
- added link bucket_cyl_barrel, mass 110; visual box size=0.114 0.095 0.076; visual box size=0.114 0.095 0.076
- added link bucket_cyl_rod, mass 55; visual cylinder length=0.19 radius=0.07125; visual cylinder length=0.807955 radius=0.05225
- added link bucket_hlink, mass 50; visual box size=0.12 0.28 0.07; visual box size=0.74 0.03 0.11
- added link bucket_idler, mass 45; visual box size=0.56 0.03 0.09; visual box size=0.56 0.03 0.09
- link boom: mass 1800 -> 1630; geometry collision box size=1.215281 0.46 0.38; collision box size=1.678246 0.55 0.6
- link bucket: mass 750 -> 700; geometry collision box size=0.335261 1.2 0.06; collision box size=0.428019 1.2 0.06
- link left_sprocket: geometry visual box size=0.1 0.64 0.8075; visual box size=0.12 0.64 0.05
- link right_sprocket: geometry visual box size=0.1 0.64 0.8075; visual box size=0.12 0.64 0.05
- link stick: mass 900 -> 780; geometry collision box size=1 0.45 0.49; collision box size=2 0.45 0.38
- link undercarriage: mass 8000 -> 7740; geometry collision box size=2.2 1.78 0.5; collision box size=3.22 0.34 0.71
- link upper_structure: mass 9000 -> 8760; geometry collision box size=0.28 0.05 0.52; collision box size=0.28 0.05 0.52
Joints:
- added joint arm_cyl_barrel_joint: type revolute, parent boom, child arm_cyl_barrel, origin xyz=3.7 0 2.65 rpy=0 0.628981 0, axis 0 -1 0, limit lower=-0.0496286022 upper=0.0496286022 effort=10000000 velocity=0.067061
- added joint arm_cyl_rod_joint: type revolute, parent stick, child arm_cyl_rod, origin xyz=-0.3 0 0.06 rpy=0 -4.107612 0, axis 0 -1 0, limit lower=-1.1746286 upper=1.1746286 effort=10000000 velocity=0.717061
- added joint boom_cyl_barrel_joint: type revolute, parent upper_structure, child boom_cyl_barrel, origin xyz=1.2 -0.09 0.4 rpy=0 -0.571978 0, axis 0 -1 0, limit lower=-0.928286908 upper=0.928286908 effort=10000000 velocity=0.575792
- added joint boom_cyl_rod_joint: type revolute, parent boom, child boom_cyl_rod, origin xyz=1.54 0 0.53 rpy=0 -3.663571 0, axis 0 -1 0, limit lower=-0.0619130916 upper=0.0619130916 effort=10000000 velocity=0.074208
- added joint bucket_cyl_barrel_joint: type revolute, parent stick, child bucket_cyl_barrel, origin xyz=0.17 0 0.3 rpy=0 -0.057422 0, axis 0 -1 0, limit lower=-0.0562207505 upper=0.0562207505 effort=10000000 velocity=0.074489
- added joint bucket_cyl_rod_joint: type revolute, parent bucket_idler, child bucket_cyl_rod, origin xyz=0.47 0 0 rpy=0 -1.744026 0, axis 0 -1 0, limit lower=-0.75551559 upper=0.75551559 effort=10000000 velocity=0.548587
- added joint bucket_hlink_joint: type revolute, parent bucket, child bucket_hlink, origin xyz=0.07 0 0.29 rpy=0 -2.920075 0, axis 0 -1 0, limit lower=-1.21877538 upper=1.21877538 effort=10000000 velocity=0.862661
- added joint bucket_idler_joint: type revolute, parent stick, child bucket_idler, origin xyz=2.36 0 0.04 rpy=0 -1.454989 0, axis 0 -1 0, limit lower=-0.791636341 upper=0.791636341 effort=10000000 velocity=0.573075

File: assets/heavy_machines/motor_grader/motor_grader.urdf (robot description, URDF)
Before this commit: robot motor_grader, 22 links, 21 joints
Links:
- link rear_frame: geometry collision box size=0.18 1.3 0.6; collision box size=0.25 0.7 0.45
Joints:
- joint blade_rotate_joint: limit lower=-1.4001 upper=1.4001 effort=10000000 velocity=0.25 -> lower=-1.22183048 upper=1.22183048 effort=10000000 velocity=0.25

File: assets/heavy_machines/wheeled_excavator/wheeled_excavator.urdf (robot description, URDF)
Before this commit: robot wheeled_excavator, 18 links, 17 joints
Links:
- link boom: geometry collision box size=2.657536 0.46 0.5; collision box size=2.773536 0.52 0.62
- link stick_cylinder_rod: geometry visual cylinder length=0.2 radius=0.09; visual cylinder length=1.72 radius=0.065
- link upper_structure: geometry collision box size=0.55 0.856507 1; collision box size=0.55 0.856507 1
Joints:
- joint stick_cylinder_joint: limit lower=-2.8704416 upper=-0.574682617 effort=10000000 velocity=0.748625 -> lower=-2.87272413 upper=-0.61716529 effort=10000000 velocity=0.751699
- joint stick_joint: limit lower=-1.3001 upper=0.8001 effort=10000000 velocity=0.65 -> lower=-1.2501 upper=0.8001 effort=10000000 velocity=0.65
